Commit message: 但是一切都不会放弃

File: chaining_package/ENV/3d_asset/3d_model/kuka_grasp/blue_block.urdf (robot description, URDF)
Before this commit: robot block_2, 1 links, 0 joints
Links:
- removed link block_2_base_link
- added link block_5_base_link, mass 0.02; collision box size=0.05 0.05 0.05; visual box size=0.05 0.05 0.05
